Commit message: Apparently urdf is flawed (IVAN FIX IT!)

File: src/test_urdf_v2/config/ArmURDF2.ros2_control.xacro (robot description, xacro)
@@ -50,32 +50,4 @@
                 <state_interface name="velocity"/>
             </joint>
-            <joint name="joint_7_1">
-                <command_interface name="position"/>
-                <state_interface name="position">
-                  <param name="initial_value">${initial_positions['joint_7_1']}</param>
-                </state_interface>
-                <state_interface name="velocity"/>
-            </joint>
-            <joint name="joint_9_1">
-                <command_interface name="position"/>
-                <state_interface name="position">
-                  <param name="initial_value">${initial_positions['joint_9_1']}</param>
-                </state_interface>
-                <state_interface name="velocity"/>
-            </joint>
-            <joint name="joint_7_2">
-                <command_interface name="position"/>
-                <state_interface name="position">
-                  <param name="initial_value">${initial_positions['joint_7_2']}</param>
-                </state_interface>
-                <state_interface name="velocity"/>
-            </joint>
-            <joint name="joint_9_2">
-                <command_interface name="position"/>
-                <state_interface name="position">
-                  <param name="initial_value">${initial_positions['joint_9_2']}</param>
-                </state_interface>
-                <state_interface name="velocity"/>
-            </joint>
             <joint name="joint_8_1">
                 <command_interface name="position"/>

Commit message: removed gripper planning group (sorry Ivan)

File: src/test_urdf_v2/config/ArmURDF2.ros2_control.xacro (robot description, xacro)
@@ -50,18 +50,4 @@
                 <state_interface name="velocity"/>
             </joint>
-            <joint name="joint_8_1">
-                <command_interface name="position"/>
-                <state_interface name="position">
-                  <param name="initial_value">${initial_positions['joint_8_1']}</param>
-                </state_interface>
-                <state_interface name="velocity"/>
-            </joint>
-            <joint name="joint_8_2">
-                <command_interface name="position"/>
-                <state_interface name="position">
-                  <param name="initial_value">${initial_positions['joint_8_2']}</param>
-                </state_interface>
-                <state_interface name="velocity"/>
-            </joint>
         </ros2_control>
     </xacro:macro>
