Commit message: Feat: get localization working with robot

File: src/ros2_rover/rover_description/robots/rover.urdf.xacro (robot description, xacro)
@@ -181,5 +181,5 @@
     </xacro:sensor_imu>
     <xacro:sensor_asus_xtion prefix="camera" parent="base_link">
-        <origin xyz="0.215 0 0.065" rpy="0 0.5 0"/>
+        <origin xyz="0.215 0 0.065" rpy="0 0 4.71238898"/>
         <!-- <origin xyz="0.212 0 0.065" rpy="0 0 0"/> -->
     </xacro:sensor_asus_xtion>

Commit message: fix: navigation tuning

File: src/ros2_rover/rover_description/robots/rover.urdf.xacro (robot description, xacro)
@@ -181,5 +181,5 @@
     </xacro:sensor_imu>
     <xacro:sensor_asus_xtion prefix="camera" parent="base_link">
-        <origin xyz="0.215 0 0.065" rpy="0 0 4.71238898"/>
+        <origin xyz="0.26 0 0.11" rpy="0 0 0"/>
         <!-- <origin xyz="0.212 0 0.065" rpy="0 0 0"/> -->
     </xacro:sensor_asus_xtion>
