Commit message: fix: use left camera

File: src/rover_description/robots/circ.urdf.xacro (robot description, xacro)
@@ -3,5 +3,5 @@
   <link name="base_link"/>
   <link name="lidar_link"/>
-  <link name="camera_link"/>
+  <link name="zed_left_frame_link"/>
   <link name="gps_link"/>
   <joint name="lidar_joint" type="fixed">
@@ -10,8 +10,8 @@
     <origin xyz="0.14 0.115 0.03 " rpy="0 0 0"/>
   </joint>
-  <joint name="camera_joint" type="fixed">
+  <joint name="zed_left_frame_joint" type="fixed">
     <parent link="base_link"/>
-    <child link="camera_link"/>
-    <origin xyz="-0.15 -0.1 0.87 " rpy="0 -0.523599 0"/>
+    <child link="zed_left_frame_link"/>
+    <origin xyz="-0.15 -0.16 0.87 " rpy="0 -0.523599 0"/>
   </joint>
   <joint name="gps_joint" type="fixed">

Commit message: fix: imu fixes

File: src/rover_description/robots/circ.urdf.xacro (robot description, xacro)
@@ -5,4 +5,5 @@
   <link name="zed_left_frame_link"/>
   <link name="gps_link"/>
+  <link name="zed_imu_link"/>
   <joint name="lidar_joint" type="fixed">
     <parent link="base_link"/>
@@ -20,3 +21,8 @@
     <origin xyz="0.0 0.0 0.0 " rpy="0 0 0"/>
   </joint>
+  <joint name="zed_imu_joint" type="fixed">
+    <parent link="zed_left_frame_link"/>
+    <child link="zed_imu_link"/>
+    <origin xyz="0.023061 0.00226 0.002 " rpy="0.00369745 -0.00188104  0.00311351"/>
+  </joint>
 </robot>

Commit message: fix: localization fixes

File: src/rover_description/robots/circ.urdf.xacro (robot description, xacro)
@@ -14,5 +14,5 @@
     <parent link="base_link"/>
     <child link="zed_left_frame_link"/>
-    <origin xyz="-0.15 -0.16 0.87 " rpy="0 -0.523599 0"/>
+    <origin xyz="-0.05 -0.15 0.83 " rpy="0 0.523599 0"/>
   </joint>
   <joint name="gps_joint" type="fixed">

Commit message: current changes

File: src/rover_description/robots/circ.urdf.xacro (robot description, xacro)
@@ -9,10 +9,10 @@
     <parent link="base_link"/>
     <child link="lidar_link"/>
-    <origin xyz="0.14 0.115 0.03 " rpy="0 0 0"/>
+    <origin xyz="0.14 -0.115 0.03 " rpy="0 0 0"/>
   </joint>
   <joint name="zed_left_frame_joint" type="fixed">
     <parent link="base_link"/>
     <child link="zed_left_frame_link"/>
-    <origin xyz="-0.05 -0.15 0.83 " rpy="0 0.523599 0"/>
+    <origin xyz="-0.05 0.15 0.83 " rpy="0 0.523599 0"/>
   </joint>
   <joint name="gps_joint" type="fixed">

Commit message: last commit

File: src/rover_description/robots/circ.urdf.xacro (robot description, xacro)
@@ -19,5 +19,5 @@
     <parent link="base_link"/>
     <child link="gps_link"/>
-    <origin xyz="0.0 0.0 0.0 " rpy="0 0 0"/>
+    <origin xyz="0.08 0.0 0.0 " rpy="0 0 0"/>
   </joint>
   <joint name="zed_imu_joint" type="fixed">
